File: board/v3_1/power-meter-v3_1.kicad_pcb (KiCad board)
At the start: 2 copper layers, 52.9 x 30.6 mm, 50 parts, among them J1 Screw_Terminal_01x04, J2 Screw_Terminal_01x02, J4 Conn_01x03, J5 Conn_01x02_Pin, U1 ADM2486, U2 FM24C64B, U3 INA228, U4 ATtiny1624-SS, U5 L78L05_TO92, U7 L78L05_TO92

Commit message: minor schematic updates
Parts:
- C7: value C_Small -> ?
- PS1: value RO-0505S -> B1212S
Connections:
- net VBUS renamed /VBUS
